File: LMX_PLL_HW/LMX2332V01.kicad_sch (KiCad schematic)
At the start: 56 parts, among them J1 142-0701-201, J2 Conn_01x04_Male, J3 Screw_Terminal_01x02, U1 Z-CommV440, U2 LMX2332, U3 ToyocomTCXO, U4 TPS784-Q1, U5 TPS784-Q1

Commit message: As sent out to OshPark. Using KiCad 6.0.
As sent out to OshPark. Using KiCad 6.0.
Parts:
- removed U1: Z-CommV440, LMX_PLL_HW:Z-CommVCO, symbol LMX2332V01-rescue:Z-CommV440-DB_KiCad
- added 3V0, 5V0, VCont1: TestPoint, TestPoint:TestPoint_THTPad_D2.0mm_Drill1.0mm, symbol Connector:TestPoint
- added U1: Z-CommV440V2, LMX_PLL_HW:ZCommVCO, symbol DB_KiCad:Z-CommV440V2
- C1: footprint Capacitors_SMD:C_0805_HandSoldering -> Capacitor_SMD:C_0805_2012Metric_Pad1.15x1.40mm_HandSolder
- CLK1: renamed from TP2; footprint TestPoint:TestPoint_THTPad_1.0x1.0mm_Drill0.5mm -> TestPoint:TestPoint_THTPad_D2.0mm_Drill1.0mm
- D3: renamed from TP4; footprint TestPoint:TestPoint_THTPad_1.0x1.0mm_Drill0.5mm -> TestPoint:TestPoint_THTPad_D2.0mm_Drill1.0mm
- FoLD1: renamed from TP3; footprint TestPoint:TestPoint_THTPad_1.0x1.0mm_Drill0.5mm -> TestPoint:TestPoint_THTPad_D2.0mm_Drill1.0mm
- GND1: renamed from TP5; footprint TestPoint:TestPoint_THTPad_1.0x1.0mm_Drill0.5mm -> TestPoint:TestPoint_THTPad_D2.0mm_Drill1.0mm
- J1: footprint JOHNSON_142-0701-201 -> LMX_PLL_HW:JOHNSON_142-0701-201
- J2: value Conn_01x04_Male -> Serial I/O; footprint Connector_JST:JST_SH_SM04B-SRSS-TB_1x04-1MP_P1.00mm_Horizontal -> Connector_JST:JST_PH_B4B-PH-K_1x04_P2.00mm_Vertical
- LE1: renamed from TP1; footprint TestPoint:TestPoint_THTPad_1.0x1.0mm_Drill0.5mm -> TestPoint:TestPoint_THTPad_D2.0mm_Drill1.0mm
Connections:
- net GND: now also J2.1 (Pin_1), U1.4 (GND); no longer J2.4 (Pin_4)
- net at CLK1.1, U2.11 (Clock): now also J2.2 (Pin_2); no longer J2.3 (Pin_3)
- net at D3.1, U2.12 (Data): now also J2.3 (Pin_3); no longer J2.2 (Pin_2)
- net at LE1.1, U2.13 (LE): now also J2.4 (Pin_4); no longer J2.1 (Pin_1)
- net at C3.1, R1.1: now also U1.1 (Vt)
- net at R3.2: now also U1.2 (RFOut)
- net at U3.5 (VCont): now also VCont1.1
- net at C6.1, C7.1, D1.2 (A)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: now also 5V0.1
- net at C10.1, C8.1, D2.2 (A)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: now also 3V0.1
- net +5V: no longer names the net of C12.1, C13.1, C14.1, C15.1, R19.2, U2.1 (Vcc), U2.19 (Vp2), U2.2 (Vp1), U2.20 (Vcc)
- net +5V: now also U1.3 (Vcc)
- net VCC: no longer names the net of C11.1, C5.1, C9.1, FB1.1, U4.1 (VIN), U4.3 (EN), U5.1 (VIN), U5.3 (EN)
Other:
- note added: "[] Add larger DNP in parallel w/ C1 [] Add SMA monitor port at U3 RF Out"
- moved on the sheet: J2
