File: LMX_PLL_HW/LMX2332V01.kicad_sch (KiCad schematic)
At the start: 59 parts, among them J1 142-0701-201, J2 Serial I/O, J3 Screw_Terminal_01x02, U1 Z-CommV440V2, U2 LMX2332, U3 ToyocomTCXO, U4 TPS784-Q1, U5 TPS784-Q1

Commit message: Update 2023-06-22
Cleanup
Other:
- note added: "[] Add larger DNP in parallel w/ C1 [] Add SMA monitor port at U3 RF Out [] Footpring for TCXO needs correcting. Pin 5/8 are swapped [] Spin LMX/VCO to improve routing of Fin/DoRF"
- note removed: "[] Add larger DNP in parallel w/ C1 [] Add SMA monitor port at U3 RF Out"
Changed lines of the file:
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@@
     (stroke (width 0) (type solid) (color 0 0 0 0))
   )
-  (text "[] Add larger DNP in parallel w/ C1\n[] Add SMA monitor port at U3 RF Out\n"
-    (at 96.52 240.03 0)
+  (text "[] Add larger DNP in parallel w/ C1\n[] Add SMA monitor port at U3 RF Out\n[] Footpring for TCXO needs correcting. Pin 5/8 are swapped\n[] Spin LMX/VCO to improve routing of Fin/DoRF\n"
+    (at 96.52 243.84 0)
     (effects (font (size 1.27 1.27)) (justify left bottom))
   )
